Commit message: Added depth camera

File: robots/hand.gazebo.xacro (robot description, xacro)
@@ -2,4 +2,46 @@
 <robot xmlns:xacro="http://www.ros.org/wiki/xacro" name="panda">
 	<gazebo reference="${ns}_hand"/>
+	<gazebo reference="${ns}_camera_link">
+		<sensor name="${ns}_camera" type="depth">
+			<pose>0 0 0 0 0 0</pose>
+			<update_rate>20</update_rate>
+			<camera>
+				<horizontal_fov>1.047198</horizontal_fov>
+				<image>
+				  <width>640</width>
+				  <height>480</height>
+				  <format>R8G8B8</format>
+				</image>
+				<clip>
+				  <near>0.01</near>
+				  <far>5.0</far>
+				</clip>
+			</camera>
+			<plugin name="${ns}_camera_controller" filename="libgazebo_ros_openni_kinect.so">
+				<baseline>0.2</baseline>
+				<alwaysOn>true</alwaysOn>
+				<updateRate>0</updateRate>
+				<cameraName>camera_ir</cameraName>
+				<imageTopicName>/camera/color/image_raw</imageTopicName>
+				<cameraInfoTopicName>/camera/color/camera_info</cameraInfoTopicName>
+				<depthImageTopicName>/camera/depth/image_raw</depthImageTopicName>
+				<depthImageInfoTopicName>/camera/depth/camera_info</depthImageInfoTopicName>
+				<pointCloudTopicName>/camera/depth/points</pointCloudTopicName>
+				<frameName>${ns}_camera_link_optical</frameName>
+				<pointCloudCutoff>0.01</pointCloudCutoff>
+				<pointCloudCutoffMax>5.0</pointCloudCutoffMax>
+				<distortionK1>0</distortionK1>
+				<distortionK2>0</distortionK2>
+				<distortionK3>0</distortionK3>
+				<distortionT1>0</distortionT1>
+				<distortionT2>0</distortionT2>
+				<CxPrime>0</CxPrime>
+				<Cx>0</Cx>
+				<Cy>0</Cy>
+				<focalLength>0</focalLength>
+				<hackBaseline>0</hackBaseline>
+			</plugin>
+		</sensor>
+	</gazebo>
 	<gazebo reference="${ns}_leftfinger"/>
 	<gazebo reference="${ns}_rightfinger"/>

File: robots/hand.xacro (robot description, xacro)
@@ -2,4 +2,5 @@
 <robot xmlns:xacro="http://www.ros.org/wiki/xacro" name="hand">
   <xacro:macro name="hand" params="connected_to:='' ns:='' rpy:='0 0 0' xyz:='0 0 0' ">
+	<xacro:property name="camera_link" value="0.03" /> <!-- Size of square 'camera' box -->
     <xacro:unless value="${connected_to == ''}">
       <joint name="${ns}_hand_joint" type="fixed">
@@ -36,4 +37,40 @@
       </collision>
     </link>
+	<!-- Camera -->
+	<link name="${ns}_camera_link">
+	  <collision>
+	    <origin xyz="0 0 0" rpy="0 0 0"/>
+	    <geometry>
+	  <box size="${camera_link} ${camera_link} ${camera_link}"/>
+	    </geometry>
+	  </collision>
+	  <visual>
+	    <origin xyz="0 0 0" rpy="0 0 0"/>
+	    <geometry>
+	  <box size="${camera_link} ${camera_link} ${camera_link}"/>
+	    </geometry>
+	  </visual>
+	  <inertial>
+	    <mass value="1e-5" />
+	    <origin xyz="0 0 0" rpy="0 0 0"/>
+	    <inertia ixx="1e-6" ixy="0" ixz="0" iyy="1e-6" iyz="0" izz="1e-6" />
+	  </inertial>
+	</link>
+	<joint name="${ns}_camera_joint" type="fixed">
+	  <axis xyz="0 0 0" />
+	  <origin xyz="0.04 0 0.05" rpy="${pi} ${-pi/2} 0"/>
+	  <parent link="${ns}_hand"/>
+	  <child link="${ns}_camera_link"/>
+	</joint>
+	<joint name="camera_optical_joint" type="fixed">
+	  <!-- these values have to be these values otherwise the gazebo camera
+	      image won't be aligned properly with the frame it is supposedly
+	      originating from -->
+	  <origin xyz="0 0 0" rpy="${-pi/2} 0 ${-pi/2}"/>
+	  <parent link="${ns}_camera_link"/>
+	  <child link="${ns}_camera_link_optical"/>
+	</joint>
+	<link name="${ns}_camera_link_optical">
+	</link>
     <link name="${ns}_leftfinger">
       <inertial>

Commit message: Add force/torque sensors

File: robots/hand.gazebo.xacro (robot description, xacro)
@@ -46,4 +46,26 @@
 	<gazebo reference="${ns}_leftfinger"/>
 	<gazebo reference="${ns}_rightfinger"/>
+	<gazebo reference="${ns}_ft_leftfinger"/>
+	<gazebo reference="${ns}_ft_rightfinger"/>
+	<gazebo reference="${ns}_ft_joint_1">
+    	<provideFeedback>true</provideFeedback>
+	</gazebo>
+	<gazebo>
+		<plugin name="ft_left_sensor" filename="libgazebo_ros_ft_sensor.so">
+		    <updateRate>100.0</updateRate>
+		    <topicName>/ft_left_sensor</topicName>
+		    <jointName>${ns}_ft_joint_1</jointName>
+		</plugin>
+	</gazebo>
+	<gazebo reference="${ns}_ft_joint_2">
+    	<provideFeedback>true</provideFeedback>
+	</gazebo>
+	<gazebo>
+		<plugin name="ft_right_sensor" filename="libgazebo_ros_ft_sensor.so">
+		    <updateRate>100.0</updateRate>
+		    <topicName>/ft_right_sensor</topicName>
+		    <jointName>${ns}_ft_joint_2</jointName>
+		</plugin>
+	</gazebo>
 	<transmission name="${ns}_finger_joint1_trans">
     <type>transmission_interface/SimpleTransmission</type>

File: robots/hand.xacro (robot description, xacro)
@@ -3,4 +3,5 @@
   <xacro:macro name="hand" params="connected_to:='' ns:='' rpy:='0 0 0' xyz:='0 0 0' ">
 	<xacro:property name="camera_link" value="0.03" /> <!-- Size of square 'camera' box -->
+	<xacro:property name="ft_link" value="0.01" /> <!-- Size of square 'force_torque' box -->
     <xacro:unless value="${connected_to == ''}">
       <joint name="${ns}_hand_joint" type="fixed">
@@ -37,40 +38,40 @@
       </collision>
     </link>
-	<!-- Camera -->
-	<link name="${ns}_camera_link">
-	  <collision>
-	    <origin xyz="0 0 0" rpy="0 0 0"/>
-	    <geometry>
-	  <box size="${camera_link} ${camera_link} ${camera_link}"/>
-	    </geometry>
-	  </collision>
-	  <visual>
-	    <origin xyz="0 0 0" rpy="0 0 0"/>
-	    <geometry>
-	  <box size="${camera_link} ${camera_link} ${camera_link}"/>
-	    </geometry>
-	  </visual>
-	  <inertial>
-	    <mass value="1e-5" />
-	    <origin xyz="0 0 0" rpy="0 0 0"/>
-	    <inertia ixx="1e-6" ixy="0" ixz="0" iyy="1e-6" iyz="0" izz="1e-6" />
-	  </inertial>
-	</link>
-	<joint name="${ns}_camera_joint" type="fixed">
-	  <axis xyz="0 0 0" />
-	  <origin xyz="0.04 0 0.05" rpy="${pi} ${-pi/2} 0"/>
-	  <parent link="${ns}_hand"/>
-	  <child link="${ns}_camera_link"/>
-	</joint>
-	<joint name="camera_optical_joint" type="fixed">
-	  <!-- these values have to be these values otherwise the gazebo camera
-	      image won't be aligned properly with the frame it is supposedly
-	      originating from -->
-	  <origin xyz="0 0 0" rpy="${-pi/2} 0 ${-pi/2}"/>
-	  <parent link="${ns}_camera_link"/>
-	  <child link="${ns}_camera_link_optical"/>
-	</joint>
-	<link name="${ns}_camera_link_optical">
-	</link>
+		<!-- Camera -->
+		<link name="${ns}_camera_link">
+			<collision>
+			  <origin xyz="0 0 0" rpy="0 0 0"/>
+			  <geometry>
+			<box size="${camera_link} ${camera_link} ${camera_link}"/>
+			  </geometry>
+			</collision>
+			<visual>
+			  <origin xyz="0 0 0" rpy="0 0 0"/>
+			  <geometry>
+			<box size="${camera_link} ${camera_link} ${camera_link}"/>
+			  </geometry>
+			</visual>
+			<inertial>
+			  <mass value="1e-5" />
+			  <origin xyz="0 0 0" rpy="0 0 0"/>
+			  <inertia ixx="1e-6" ixy="0" ixz="0" iyy="1e-6" iyz="0" izz="1e-6" />
+			</inertial>
+		</link>
+		<joint name="${ns}_camera_joint" type="fixed">
+			<axis xyz="0 0 0" />
+			<origin xyz="0.04 0 0.05" rpy="${pi} ${-pi/2} 0"/>
+			<parent link="${ns}_hand"/>
+			<child link="${ns}_camera_link"/>
+		</joint>
+		<joint name="camera_optical_joint" type="fixed">
+			<!-- these values have to be these values otherwise the gazebo camera
+			    image won't be aligned properly with the frame it is supposedly
+			    originating from -->
+			<origin xyz="0 0 0" rpy="${-pi/2} 0 ${-pi/2}"/>
+			<parent link="${ns}_camera_link"/>
+			<child link="${ns}_camera_link_optical"/>
+		</joint>
+		<link name="${ns}_camera_link_optical">
+		</link>
     <link name="${ns}_leftfinger">
       <inertial>
@@ -131,4 +132,54 @@
       <limit effort="20" lower="-0.001" upper="0.04" velocity="0.3"/>
     </joint>
+		<link name="${ns}_ft_leftfinger">
+			<collision>
+			  <origin xyz="0 0 0" rpy="0 0 0"/>
+			  <geometry>
+			<box size="${ft_link} ${ft_link} ${ft_link}"/>
+			  </geometry>
+			</collision>
+			<visual>
+			  <origin xyz="0 0 0" rpy="0 0 0"/>
+			  <geometry>
+			<box size="${ft_link} ${ft_link} ${ft_link}"/>
+			  </geometry>
+			</visual>
+			<inertial>
+			  <mass value="1e-5" />
+			  <origin xyz="0 0 0" rpy="0 0 0"/>
+			  <inertia ixx="1e-6" ixy="0" ixz="0" iyy="1e-6" iyz="0" izz="1e-6" />
+			</inertial>
+		</link>
+		<link name="${ns}_ft_rightfinger">
+			<collision>
+			  <origin xyz="0 0 0" rpy="0 0 0"/>
+			  <geometry>
+			<box size="${ft_link} ${ft_link} ${ft_link}"/>
+			  </geometry>
+			</collision>
+			<visual>
+			  <origin xyz="0 0 0" rpy="0 0 0"/>
+			  <geometry>
+			<box size="${ft_link} ${ft_link} ${ft_link}"/>
+			  </geometry>
+			</visual>
+			<inertial>
+			  <mass value="1e-5" />
+			  <origin xyz="0 0 0" rpy="0 0 0"/>
+			  <inertia ixx="1e-6" ixy="0" ixz="0" iyy="1e-6" iyz="0" izz="1e-6" />
+			</inertial>
+		</link>
+		<joint name="${ns}_ft_joint_1" type="revolute">
+		    <parent link="${ns}_leftfinger"/>
+		    <child link="${ns}_ft_leftfinger"/>
+		    <origin xyz="0 -0.005 0.06" rpy="0 0 0"/>
+				<limit velocity="6.5" effort="1000" lower="0" upper="0" />
+		  </joint>
+    <joint name="${ns}_ft_joint_2" type="revolute">
+      <parent link="${ns}_rightfinger"/>
+      <child link="${ns}_ft_rightfinger"/>
+      <origin xyz="0 0.005 0.06" rpy="0 0 ${pi}"/>
+			<limit velocity="6.5" effort="1000" lower="0" upper="0" />
+    </joint>
   </xacro:macro>
 </robot>
