Commit message: Fix sensors position

File: robots/hand.xacro (robot description, xacro)
@@ -173,5 +173,5 @@
 		    <parent link="${ns}_leftfinger"/>
 		    <child link="${ns}_ft_leftfinger"/>
-		    <origin xyz="0 -0.005 0.06" rpy="0 0 0"/>
+		    <origin xyz="0 0.005 0.06" rpy="0 0 0"/>
 				<limit velocity="6.5" effort="1000" lower="0" upper="0" />
 		  </joint>
@@ -179,5 +179,5 @@
       <parent link="${ns}_rightfinger"/>
       <child link="${ns}_ft_rightfinger"/>
-      <origin xyz="0 0.005 0.06" rpy="0 0 ${pi}"/>
+      <origin xyz="0 -0.005 0.06" rpy="0 0 ${pi}"/>
 			<limit velocity="6.5" effort="1000" lower="0" upper="0" />
     </joint>
